Commit message: add_pan_tilt_config

File: src/pan_tilt_urdf/urdf/pan_tilt_simple.urdf (robot description, URDF)
Before this commit: robot simple_pan_tilt, 2 links, 1 joints
Links:
- removed link top_servo_link
- added link top_pan_link; collision box size=0.033 0.05 0.065; visual box size=0.033 0.05 0.065
- added link top_tilt_link; collision box size=0.025 0.078 0.043; visual box size=0.025 0.078 0.043
Joints:
- removed joint base_to_top_servo
- added joint pan_joint: type revolute, parent base_link, child top_pan_link, origin xyz=0.011 0.0 0.0725 rpy=0 0 0, axis 0 0 1, limit lower=-1.57 upper=1.57 effort=1000.0 velocity=0.5
- added joint tilt_joint: type revolute, parent top_pan_link, child top_tilt_link, origin xyz=0 0 0.016 rpy=0 0 3.142, axis 0 1 0, limit lower=-1.57 upper=1.57 effort=1000.0 velocity=0.5
